Commit message: Added new world

File: parol6_moveit2_config/config/parol6.urdf.xacro (robot description, xacro)
@@ -17,5 +17,5 @@
     <!-- World fixed joint-->
     <joint name="world_fixed" type="fixed">
-        <origin xyz="0 0 0" rpy="0 0 0"/>
+        <origin xyz="-0.526520 -1.121150 0.7998145" rpy="0 0 0"/>
         <parent link="world"/>
         <child link="base_link"/>
