Commit message: Added launch files

File: parol6_description/urdf/parol6.urdf.xacro (robot description, xacro)
@@ -16,14 +16,18 @@
         <origin xyz="0 0 0" rpy="0 0 0" />
         <geometry>
-          <mesh filename="package://parol6_description/meshes/base_link.dae" />
-        </geometry>
-      </visual>
-      <collision>
-        <origin xyz="0 0 0" rpy="0 0 0" />
-        <geometry>
-          <mesh filename="package://parol6_description/meshes/base_link.dae" />
-        </geometry>
-      </collision>
-    </link>
+          <mesh filename="file:///home/azif/projetcs/parol6/parol6_description/meshes/base_link.dae"/>
+        </geometry>
+      </visual>
+      <collision>
+        <origin xyz="0 0 0" rpy="0 0 0" />
+        <geometry>
+          <mesh filename="file:///home/azif/projetcs/parol6/parol6_description/meshes/base_link.dae"/>
+        </geometry>
+      </collision>
+    </link>
+    <!-- <gazebo reference="base_link">
+      <material>Gazebo/Orange</material>
+      <turnGravityOff>false</turnGravityOff>
+    </gazebo> -->
     <link name="L1">
       <inertial>
@@ -36,11 +40,11 @@
         <origin xyz="0 0 0" rpy="0 0 0" />
         <geometry>
-          <mesh filename="package://parol6_description/meshes/L1.dae" />
-        </geometry>
-      </visual>
-      <collision>
-        <origin xyz="0 0 0" rpy="0 0 0" />
-        <geometry>
-          <mesh filename="package://parol6_description/meshes/L1.dae" />
+          <mesh filename="file:///home/azif/projetcs/parol6/parol6_description/meshes/L1.dae"/>
+        </geometry>
+      </visual>
+      <collision>
+        <origin xyz="0 0 0" rpy="0 0 0" />
+        <geometry>
+          <mesh filename="file:///home/azif/projetcs/parol6/parol6_description/meshes/L1.dae"/>
         </geometry>
       </collision>
@@ -63,11 +67,11 @@
         <origin xyz="0 0 0" rpy="0 0 0" />
         <geometry>
-          <mesh filename="package://parol6_description/meshes/L2.dae" />
-        </geometry>
-      </visual>
-      <collision>
-        <origin xyz="0 0 0" rpy="0 0 0" />
-        <geometry>
-          <mesh filename="package://parol6_description/meshes/L2.dae" />
+          <mesh filename="file:///home/azif/projetcs/parol6/parol6_description/meshes/L2.dae"/>
+        </geometry>
+      </visual>
+      <collision>
+        <origin xyz="0 0 0" rpy="0 0 0" />
+        <geometry>
+          <mesh filename="file:///home/azif/projetcs/parol6/parol6_description/meshes/L2.dae"/>
         </geometry>
       </collision>
@@ -90,11 +94,11 @@
         <origin xyz="0 0 0" rpy="0 0 0" />
         <geometry>
-          <mesh filename="package://parol6_description/meshes/L3.dae" />
-        </geometry>
-      </visual>
-      <collision>
-        <origin xyz="0 0 0" rpy="0 0 0" />
-        <geometry>
-          <mesh filename="package://parol6_description/meshes/L3.dae" />
+          <mesh filename="file:///home/azif/projetcs/parol6/parol6_description/meshes/L3.dae"/>
+        </geometry>
+      </visual>
+      <collision>
+        <origin xyz="0 0 0" rpy="0 0 0" />
+        <geometry>
+          <mesh filename="file:///home/azif/projetcs/parol6/parol6_description/meshes/L3.dae"/>
         </geometry>
       </collision>
@@ -117,11 +121,10 @@
         <origin xyz="0 0 0" rpy="0 0 0" />
         <geometry>
-          <mesh filename="package://parol6_description/meshes/L4.dae"/>
-        </geometry>
-      </visual>
-      <collision>
-        <mesh filename="package://parol6_description/meshes/L4.dae"/>
-        <geometry>
-           <mesh filename="package://parol6_description/meshes/L4.dae"/>
+          <mesh filename="file:///home/azif/projetcs/parol6/parol6_description/meshes/L4.dae"/>
+        </geometry>
+      </visual>
+      <collision>
+        <geometry>
+           <mesh filename="file:///home/azif/projetcs/parol6/parol6_description/meshes/L4.dae"/>
         </geometry>
       </collision>
@@ -149,5 +152,5 @@
       <origin xyz="0 0 0" rpy="0 0 0" />
       <geometry>
-        <mesh filename="package://parol6_description/meshes/L5.dae" />
+        <mesh filename="file:///home/azif/projetcs/parol6/parol6_description/meshes/L5.dae"/>
       </geometry>
     </visual>
@@ -155,5 +158,5 @@
       <origin xyz="0 0 0" rpy="0 0 0" />
       <geometry>
-        <mesh filename="package://parol6_description/meshes/L5.dae" />
+        <mesh filename="file:///home/azif/projetcs/parol6/parol6_description/meshes/L5.dae"/>
       </geometry>
     </collision>
@@ -181,5 +184,5 @@
       <origin xyz="0 0 0" rpy="0 0 0" />
       <geometry>
-        <mesh filename="package://parol6_description/meshes/L6.dae" />
+        <mesh filename="file:///home/azif/projetcs/parol6/parol6_description/meshes/L6.dae"/>
       </geometry>
     </visual>
@@ -187,5 +190,5 @@
       <origin xyz="0 0 0" rpy="0 0 0" />
       <geometry>
-        <mesh filename="package://parol6_description/meshes/L6.dae" />
+        <mesh filename="file:///home/azif/projetcs/parol6/parol6_description/meshes/L6.dae"/>
       </geometry>
     </collision>
@@ -198,3 +201,8 @@
     <limit lower="0" upper="0" effort="0" velocity="0" />
   </joint>
+  <!-- <gazebo>
+    <plugin name="gazebo_ros_control" filename="libgazebo_ros2_control.so">
+      <robot_namespace>/</robot_namespace>
+    </plugin>
+  </gazebo> -->
 </robot>

Commit message: Added end efferctor

File: parol6_description/urdf/parol6.urdf.xacro (robot description, xacro)
@@ -184,5 +184,5 @@
       <origin xyz="0 0 0" rpy="0 0 0" />
       <geometry>
-        <mesh filename="file:///home/azif/projetcs/parol6/parol6_description/meshes/L6.dae"/>
+        <mesh filename="file:///home/azif/projetcs/parol6/parol6_description/meshes/vaccum_gripper_holder.stl"/>
       </geometry>
     </visual>
@@ -190,5 +190,5 @@
       <origin xyz="0 0 0" rpy="0 0 0" />
       <geometry>
-        <mesh filename="file:///home/azif/projetcs/parol6/parol6_description/meshes/L6.dae"/>
+        <mesh filename="file:///home/azif/projetcs/parol6/parol6_description/meshes/vaccum_gripper_holder.stl"/>
       </geometry>
     </collision>
@@ -201,8 +201,36 @@
     <limit lower="0" upper="0" effort="0" velocity="0" />
   </joint>
-  <!-- <gazebo>
-    <plugin name="gazebo_ros_control" filename="libgazebo_ros2_control.so">
-      <robot_namespace>/</robot_namespace>
-    </plugin>
-  </gazebo> -->
+  <link name="suction_gripper">
+    <visual>
+      <origin xyz="0 0 0" rpy="0 0 0"/>
+      <geometry>
+        <mesh filename="file:///home/azif/projetcs/parol6/parol6_description/meshes/vaccum_gripper.stl"/>
+      </geometry>
+    </visual>
+    <collision>
+      <origin xyz="0 0 0" rpy="0 0 0"/>
+      <geometry>
+        <mesh filename="file:///home/azif/projetcs/parol6/parol6_description/meshes/vaccum_gripper.stl"/>
+      </geometry>
+    </collision>
+    <inertial>
+      <origin xyz="0 0 0" rpy="0 0 0"/>
+      <mass value="0.01"/>
+      <inertia
+        ixx="1e-6" ixy="0" ixz="0"
+        iyy="1e-6" iyz="0"
+        izz="1e-6"/>
+    </inertial>
+  </link>
+  <joint name="J7" type="fixed">
+    <parent link="L6"/>
+    <child link="suction_gripper"/>
+    <origin xyz="0 0 0" rpy="0 0 0"/>
+  </joint>
+  <link name="tool0"/>
+  <joint name="tool0_fixed" type="fixed">
+    <parent link="suction_gripper"/>
+    <child link="tool0"/>
+    <origin xyz="0.083695 -0.000779 -0.060305" rpy="0 0 0"/>
+  </joint>
 </robot>

Commit message: Changed file structure

File: parol6_description/urdf/parol6.urdf.xacro (robot description, xacro)
@@ -1,236 +1,23 @@
-<?xml version="1.0" encoding="utf-8"?>
-<!-- This Xacro URDF was automatically created by SolidWorks to URDF Exporter!
-     Originally created by Stephen Brawner (brawner@gmail.com)
-     Commit Version: 1.6.0-4-g7f85cfe  Build Version: 1.6.7995.38578
-     Converted to Xacro by request -->
-<robot xmlns:xacro="http://wiki.ros.org/xacro"
-      name="parol6">
-    <link name="base_link">
-      <inertial>
-        <origin xyz="-0.0274562034602567 -0.00137265400595656 0.031237920982338" rpy="0 0 0" />
-        <mass value="0.812661291810144" />
-        <inertia ixx="0.00110740279540382" ixy="4.67463481205112E-05" ixz="8.47873933528831E-06"
-                iyy="0.00106582362830227" iyz="-2.6194130573118E-06" izz="0.00147883396699374" />
-      </inertial>
-      <visual>
-        <origin xyz="0 0 0" rpy="0 0 0" />
-        <geometry>
-          <mesh filename="file:///home/azif/projetcs/parol6/parol6_description/meshes/base_link.dae"/>
-        </geometry>
-      </visual>
-      <collision>
-        <origin xyz="0 0 0" rpy="0 0 0" />
-        <geometry>
-          <mesh filename="file:///home/azif/projetcs/parol6/parol6_description/meshes/base_link.dae"/>
-        </geometry>
-      </collision>
-    </link>
-    <!-- <gazebo reference="base_link">
-      <material>Gazebo/Orange</material>
-      <turnGravityOff>false</turnGravityOff>
-    </gazebo> -->
-    <link name="L1">
-      <inertial>
-        <origin xyz="0.00524529891406311 0.0289722820784871 0.0992791429452917" rpy="0 0 0" />
-        <mass value="0.644800830530233" />
-        <inertia ixx="0.00109429409029172" ixy="-6.27156874097953E-05" ixz="-5.70466862844753E-05"
-                iyy="0.00056996197700816" iyz="-0.000121686402940313" izz="0.00129487722474286" />
-      </inertial>
-      <visual>
-        <origin xyz="0 0 0" rpy="0 0 0" />
-        <geometry>
-          <mesh filename="file:///home/azif/projetcs/parol6/parol6_description/meshes/L1.dae"/>
-        </geometry>
-      </visual>
-      <collision>
-        <origin xyz="0 0 0" rpy="0 0 0" />
-        <geometry>
-          <mesh filename="file:///home/azif/projetcs/parol6/parol6_description/meshes/L1.dae"/>
-        </geometry>
-      </collision>
-    </link>
-    <joint name="J1" type="revolute">
-      <origin xyz="0 0 0" rpy="0 0 0" />
-      <parent link="base_link" />
-      <child link="L1" />
-      <axis xyz="0 0 1" />
-      <limit lower="-3.14" upper="3.14" effort="0" velocity="0" />
+<?xml version="1.0"?>
+<robot xmlns:xacro="http://www.ros.org/wiki/xacro" name="parol6">
+    <xacro:arg name="initial_positions_file" default="initial_positions.yaml" />
+    <!-- Import parol6 urdf file -->
+    <xacro:include filename="$(find parol6_description)/urdf/parol6_base.urdf.xacro" />
+    <!-- Import control_xacro -->
+    <xacro:include filename="parol6.ros2_control.xacro" />
+    <!-- <xacro:parol6_ros2_control name="FakeSystem" initial_positions_file="$(arg initial_positions_file)"/> -->
+    <xacro:parol6_ros2_control name="parol6" initial_positions_file="$(find parol6_moveit2_config)/config/initial_positions.yaml"/>
+    <gazebo>
+      <plugin name="gazebo_ros2_control" filename="libgazebo_ros2_control.so">
+        <parameters>$(find parol6_moveit2_config)/config/ros2_controllers.yaml</parameters>
+      </plugin>
+    </gazebo>
+    <!-- World -->
+    <link name="world"/>
+    <!-- World fixed joint-->
+    <joint name="world_fixed" type="fixed">
+        <origin xyz="-0.526520 -1.121150 0.7998145" rpy="0 0 0"/>
+        <parent link="world"/>
+        <child link="base_link"/>
     </joint>
-    <link name="L2">
-      <inertial>
-        <origin xyz="-0.0094181617193695 -0.0783879603613605 0.0369429741417731" rpy="0 0 0" />
-        <mass value="0.512334779399788" />
-        <inertia ixx="0.00123357482646866" ixy="3.63236238096924E-06" ixz="-3.30834557934783E-07"
-                iyy="0.000205462733796053" iyz="4.86441772103282E-07" izz="0.00132225033266162" />
-      </inertial>
-      <visual>
-        <origin xyz="0 0 0" rpy="0 0 0" />
-        <geometry>
-          <mesh filename="file:///home/azif/projetcs/parol6/parol6_description/meshes/L2.dae"/>
-        </geometry>
-      </visual>
-      <collision>
-        <origin xyz="0 0 0" rpy="0 0 0" />
-        <geometry>
-          <mesh filename="file:///home/azif/projetcs/parol6/parol6_description/meshes/L2.dae"/>
-        </geometry>
-      </collision>
-    </link>
-    <joint name="J2" type="revolute">
-      <origin xyz="0.0234207210610375 0 0.1105" rpy="-1.5707963267949 0 0" />
-      <parent link="L1" />
-      <child link="L2" />
-      <axis xyz="0 0 1" />
-      <limit lower="-1.57" upper="1.57" effort="0" velocity="0" />
-    </joint>
-    <link name="L3">
-      <inertial>
-        <origin xyz="0.0155509885239593 -0.0191127686426613 -0.00153322577917236" rpy="0 0 0" />
-        <mass value="0.550970997806044" />
-        <inertia ixx="0.00057827573271994" ixy="0.000116505232322314" ixz="-1.19955293256513E-05"
-                iyy="0.000567011676944701" iyz="1.55814255036021E-05" izz="0.000815862001506843" />
-      </inertial>
-      <visual>
-        <origin xyz="0 0 0" rpy="0 0 0" />
-        <geometry>
-          <mesh filename="file:///home/azif/projetcs/parol6/parol6_description/meshes/L3.dae"/>
-        </geometry>
-      </visual>
-      <collision>
-        <origin xyz="0 0 0" rpy="0 0 0" />
-        <geometry>
-          <mesh filename="file:///home/azif/projetcs/parol6/parol6_description/meshes/L3.dae"/>
-        </geometry>
-      </collision>
-    </link>
-    <joint name="J3" type="revolute">
-      <origin xyz="0 -0.18 0" rpy="3.1416 0 -1.5708" />
-      <parent link="L2" />
-      <child link="L3" />
-      <axis xyz="0 0 -1" />
-      <limit lower="-1.57" upper="1.57" effort="0" velocity="0" />
-    </joint>
-    <link name="L4">
-      <inertial>
-        <origin xyz="0.000947028430634433 -0.008978947112462 -0.0924798659827059" rpy="0 0 0" />
-        <mass value="0.39346362633915" />
-        <inertia ixx="0.000371672516830215" ixy="-1.05560000666389E-05" ixz="-1.56899445418326E-07"
-                iyy="0.000332364226344361" iyz="-6.10397110934672E-05" izz="0.000250606789571909" />
-      </inertial>
-      <visual>
-        <origin xyz="0 0 0" rpy="0 0 0" />
-        <geometry>
-          <mesh filename="file:///home/azif/projetcs/parol6/parol6_description/meshes/L4.dae"/>
-        </geometry>
-      </visual>
-      <collision>
-        <geometry>
-           <mesh filename="file:///home/azif/projetcs/parol6/parol6_description/meshes/L4.dae"/>
-        </geometry>
-      </collision>
-    </link>
-    <joint name="J4" type="revolute">
-      <origin xyz="0.0435 0.0 0.0" rpy="1.5708 0 3.1415" />
-      <parent link="L3" />
-      <child link="L4" />
-      <axis xyz="0 0 1" />
-      <limit lower="-1.57" upper="1.57" effort="0" velocity="0" />
-    </joint>
-    <link name="L5">
-    <inertial>
-      <origin xyz="6.7162171684676E-06 -0.00621420980825221 -0.000960871025916146" rpy="0 0 0" />
-      <mass value="0.185171777001718" />
-      <inertia
-        ixx="0.000109176748460021"
-        ixy="-1.27195013439061E-07"
-        ixz="8.4436049148633E-08"
-        iyy="8.41307588934268E-05"
-        iyz="-4.41596193640049E-07"
-        izz="0.000110629136236229" />
-    </inertial>
-    <visual>
-      <origin xyz="0 0 0" rpy="0 0 0" />
-      <geometry>
-        <mesh filename="file:///home/azif/projetcs/parol6/parol6_description/meshes/L5.dae"/>
-      </geometry>
-    </visual>
-    <collision>
-      <origin xyz="0 0 0" rpy="0 0 0" />
-      <geometry>
-        <mesh filename="file:///home/azif/projetcs/parol6/parol6_description/meshes/L5.dae"/>
-      </geometry>
-    </collision>
-  </link>
-  <joint name="J5" type="revolute">
-    <origin xyz="0 0 -0.17635" rpy="-1.5708 0 0" />
-    <parent link="L4" />
-    <child link="L5" />
-    <axis xyz="0 0 -1" />
-      <limit lower="-1.57" upper="1.57" effort="0" velocity="0" />
-  </joint>
-  <link name="L6">
-    <inertial>
-      <origin xyz="0.00632955087228015 -0.000453856352095022 -0.0554441567386594" rpy="0 0 0" />
-      <mass value="0.0703261410665101" />
-      <inertia
-        ixx="1.40276237518287E-05"
-        ixy="3.15503246005279E-07"
-        ixz="-9.28469598788221E-07"
-        iyy="1.81406721166117E-05"
-        iyz="-9.43630009030796E-07"
-        izz="2.34608103291027E-05" />
-    </inertial>
-    <visual>
-      <origin xyz="0 0 0" rpy="0 0 0" />
-      <geometry>
-        <mesh filename="file:///home/azif/projetcs/parol6/parol6_description/meshes/vaccum_gripper_holder.stl"/>
-      </geometry>
-    </visual>
-    <collision>
-      <origin xyz="0 0 0" rpy="0 0 0" />
-      <geometry>
-        <mesh filename="file:///home/azif/projetcs/parol6/parol6_description/meshes/vaccum_gripper_holder.stl"/>
-      </geometry>
-    </collision>
-  </link>
-  <joint name="J6" type="continuous">
-    <origin xyz="0 0 0" rpy="1.5708 0 0" />
-    <parent link="L5" />
-    <child link="L6" />
-    <axis xyz="0 0 -1" />
-    <limit lower="0" upper="0" effort="0" velocity="0" />
-  </joint>
-  <link name="suction_gripper">
-    <visual>
-      <origin xyz="0 0 0" rpy="0 0 0"/>
-      <geometry>
-        <mesh filename="file:///home/azif/projetcs/parol6/parol6_description/meshes/vaccum_gripper.stl"/>
-      </geometry>
-    </visual>
-    <collision>
-      <origin xyz="0 0 0" rpy="0 0 0"/>
-      <geometry>
-        <mesh filename="file:///home/azif/projetcs/parol6/parol6_description/meshes/vaccum_gripper.stl"/>
-      </geometry>
-    </collision>
-    <inertial>
-      <origin xyz="0 0 0" rpy="0 0 0"/>
-      <mass value="0.01"/>
-      <inertia
-        ixx="1e-6" ixy="0" ixz="0"
-        iyy="1e-6" iyz="0"
-        izz="1e-6"/>
-    </inertial>
-  </link>
-  <joint name="J7" type="fixed">
-    <parent link="L6"/>
-    <child link="suction_gripper"/>
-    <origin xyz="0 0 0" rpy="0 0 0"/>
-  </joint>
-  <link name="tool0"/>
-  <joint name="tool0_fixed" type="fixed">
-    <parent link="suction_gripper"/>
-    <child link="tool0"/>
-    <origin xyz="0.083695 -0.000779 -0.060305" rpy="0 0 0"/>
-  </joint>
 </robot>

Commit message: Update conveyor belt models and world files for improved integration and performance

File: parol6_description/urdf/parol6.urdf.xacro (robot description, xacro)
@@ -17,5 +17,5 @@
     <!-- World fixed joint-->
     <joint name="world_fixed" type="fixed">
-        <origin xyz="-0.526520 -1.121150 0.7998145" rpy="0 0 0"/>
+        <origin xyz="-0.526520 -1.121150 0.789815" rpy="0 0 0"/>
         <parent link="world"/>
         <child link="base_link"/>
