Commit message: Enhance conveyor belt and box spawner functionality: - Implement stepwise movement for Conveyor 2 and add soft reset for joint position. - Update box spawner plugin with improved size and mass configurations. - Introduce camera module in URDF for better integration. - Modify world file to include attach/detach plugin for enhanced interaction. - Update targets in JSON for improved robot data handling.

File: parol6_description/urdf/parol6.urdf.xacro (robot description, xacro)
@@ -6,4 +6,6 @@
     <!-- Import control_xacro -->
     <xacro:include filename="parol6.ros2_control.xacro" />
+    <xacro:include filename="$(find parol6_description)/urdf/camera_module.urdf.xacro" />
+    <xacro:intel_d435_camera parent_link="world" prefix="d435_"/>
     <!-- <xacro:parol6_ros2_control name="FakeSystem" initial_positions_file="$(arg initial_positions_file)"/> -->
     <xacro:parol6_ros2_control name="parol6" initial_positions_file="$(find parol6_moveit2_config)/config/initial_positions.yaml"/>

File: parol6_description/urdf/parol6_base.urdf.xacro (robot description, xacro)
@@ -8,8 +8,8 @@
   <link name="base_link">
       <inertial>
-        <origin xyz="-0.041184305190385045 -0.00205898100893484 0.046856881473507" rpy="0 0 0" />
-        <mass value="2.742731859859236" />
-        <inertia ixx="0.008409339977597758" ixy="0.00035498008104013193" ixz="6.43854268273456e-05"
-                iyy="0.00106582362830227" iyz="-2.6194130573118E-06" izz="0.00147883396699374" />
+<origin xyz="-0.041184305190385045 -0.00205898100893484 0.046856881473507" rpy="0 0 0" />
+        <mass value="1.0"/>
+        <inertia ixx="0.01" ixy="0.0" ixz="0.0"
+                 iyy="0.01" iyz="0.0" izz="0.01"/>
       </inertial>
       <visual>
@@ -36,7 +36,7 @@
       <inertial>
         <origin xyz="0.007867948371094665 0.043458423117730655 0.14891871441793755" rpy="0 0 0" />
-        <mass value="2.176202803039536" />
-        <inertia ixx="0.00830979574815275" ixy="-0.0004762472512681331" ixz="-0.00043319827397273435"
-                iyy="0.00056996197700816" iyz="-0.000121686402940313" izz="0.00129487722474286" />
+        <mass value="1.0"/>
+        <inertia ixx="0.01" ixy="0.0" ixz="0.0"
+                 iyy="0.01" iyz="0.0" izz="0.01"/>
       </inertial>
       <visual>
@@ -66,7 +66,7 @@
       <inertial>
         <origin xyz="-0.014127242579054249 -0.11758194054204076 0.055414461212659645" rpy="0 0 0" />
-        <mass value="1.7291298804742845" />
-        <inertia ixx="0.009367458838496387" ixy="2.7583251830485166e-05" ixz="-2.5122749243172585e-06"
-                iyy="0.000205462733796053" iyz="4.86441772103282E-07" izz="0.00132225033266162" />
+        <mass value="1.0"/>
+        <inertia ixx="0.01" ixy="0.0" ixz="0.0"
+                 iyy="0.01" iyz="0.0" izz="0.01"/>
       </inertial>
       <visual>
@@ -96,7 +96,7 @@
       <inertial>
         <origin xyz="0.02332648278593895 -0.028669152963991952 -0.00229983866875854" rpy="0 0 0" />
-        <mass value="1.8595271175953985" />
-        <inertia ixx="0.004391281345342044" ixy="0.0008847116079475719" ixz="-9.109105081666456e-05"
-                iyy="0.000567011676944701" iyz="1.55814255036021E-05" izz="0.000815862001506843" />
+        <mass value="1.0"/>
+        <inertia ixx="0.01" ixy="0.0" ixz="0.0"
+                 iyy="0.01" iyz="0.0" izz="0.01"/>
       </inertial>
       <visual>
@@ -125,8 +125,8 @@
   <link name="L4">
       <inertial>
-        <origin xyz="0.0014205426459516495 -0.013468420668693002 -0.13871979897405884" rpy="0 0 0" />
-        <mass value="1.3279397388946312" />
-        <inertia ixx="0.0028223881746794453" ixy="-8.015962550603914e-05" ixz="-1.191455163645413e-06"
-                iyy="0.000332364226344361" iyz="-6.10397110934672E-05" izz="0.000250606789571909" />
+<origin xyz="0.0014205426459516495 -0.013468420668693002 -0.13871979897405884" rpy="0 0 0" />
+        <mass value="1.0"/>
+        <inertia ixx="0.01" ixy="0.0" ixz="0.0"
+                 iyy="0.01" iyz="0.0" izz="0.01"/>
       </inertial>
       <visual>
@@ -156,11 +156,6 @@
         <origin xyz="1.00743257527014e-05 -0.009321314712378315 -0.001441306538874219" rpy="0 0 0" />
         <mass value="0.6249547473807983" />
-        <inertia
-          ixx="0.000109176748460021"
-          ixy="-1.27195013439061E-07"
-          ixz="8.4436049148633E-08"
-          iyy="8.41307588934268E-05"
-          iyz="-4.41596193640049E-07"
-          izz="0.000110629136236229" />
+        <inertia ixx="0.01" ixy="0.0" ixz="0.0"
+                 iyy="0.01" iyz="0.0" izz="0.01"/>
       </inertial>
       <visual>
@@ -191,11 +186,6 @@
         <origin xyz="0.009494326308420224 -0.000680784528142533 -0.0831662351079891" rpy="0 0 0" />
         <mass value="0.23735072609947158" />
-        <inertia
-          ixx="1.40276237518287E-05"
-          ixy="3.15503246005279E-07"
-          ixz="-9.28469598788221E-07"
-          iyy="1.81406721166117E-05"
-          iyz="-9.43630009030796E-07"
-          izz="2.34608103291027E-05" />
+        <inertia ixx="0.01" ixy="0.0" ixz="0.0"
+                 iyy="0.01" iyz="0.0" izz="0.01"/>
       </inertial>
       <visual>
@@ -236,10 +226,8 @@
       </collision>
       <inertial>
-        <origin xyz="0.0 0.0 0.0" rpy="0 0 0"/>
-        <mass value="0.03375"/>
-        <inertia
-          ixx="1e-6" ixy="0" ixz="0"
-          iyy="1e-6" iyz="0"
-          izz="1e-6"/>
+        <origin xyz="0 0 0" rpy="0 0 0"/>
+        <mass value="1.0"/>
+        <inertia ixx="0.01" ixy="0.0" ixz="0.0"
+                 iyy="0.01" iyz="0.0" izz="0.01"/>
       </inertial>
   </link>

Commit message: Changed the structure

File: parol6_description/urdf/parol6.urdf.xacro (robot description, xacro)
@@ -1,25 +1,25 @@
 <?xml version="1.0"?>
 <robot xmlns:xacro="http://www.ros.org/wiki/xacro" name="parol6">
-    <xacro:arg name="initial_positions_file" default="initial_positions.yaml" />
+  <xacro:arg name="initial_positions_file" default="initial_positions.yaml" />
     <!-- Import parol6 urdf file -->
-    <xacro:include filename="$(find parol6_description)/urdf/parol6_base.urdf.xacro" />
+  <xacro:include filename="$(find parol6_description)/urdf/parol6_base.urdf.xacro" />
     <!-- Import control_xacro -->
-    <xacro:include filename="parol6.ros2_control.xacro" />
+  <xacro:include filename="parol6.ros2_control.xacro" />
     <!-- <xacro:include filename="$(find parol6_description)/urdf/camera_module.urdf.xacro" />
     <xacro:intel_d435_camera parent_link="world" prefix="d435_"/> -->
     <!-- <xacro:parol6_ros2_control name="FakeSystem" initial_positions_file="$(arg initial_positions_file)"/> -->
-    <xacro:parol6_ros2_control name="parol6" initial_positions_file="$(find parol6_moveit2_config)/config/initial_positions.yaml"/>
-    <gazebo>
-      <plugin name="gazebo_ros2_control" filename="libgazebo_ros2_control.so">
-        <parameters>$(find parol6_moveit2_config)/config/ros2_controllers.yaml</parameters>
-      </plugin>
-    </gazebo>
+  <xacro:parol6_ros2_control name="parol6" initial_positions_file="$(find parol6_moveit2_config)/config/initial_positions.yaml"/>
+  <gazebo>
+    <plugin name="gazebo_ros2_control" filename="libgazebo_ros2_control.so">
+      <parameters>$(find parol6_moveit2_config)/config/ros2_controllers.yaml</parameters>
+    </plugin>
+  </gazebo>
     <!-- World -->
-    <link name="world"/>
+  <link name="world"/>
     <!-- World fixed joint-->
-    <joint name="world_fixed" type="fixed">
-        <origin xyz="-0.526520 -1.121150 0.789815" rpy="0 0 0"/>
-        <parent link="world"/>
-        <child link="base_link"/>
-    </joint>
+  <joint name="world_fixed" type="fixed">
+    <origin xyz="-0.526520 -1.121150 0.789815" rpy="0 0 0"/>
+    <parent link="world"/>
+    <child link="base_link"/>
+  </joint>
 </robot>

File: parol6_description/urdf/parol6_base.urdf.xacro (robot description, xacro)
@@ -61,5 +61,5 @@
       <child link="L1" />
       <axis xyz="0 0 1" />
-      <limit lower="-3.14" upper="3.14" effort="0" velocity="0" />
+      <limit lower="-3.14" upper="3.14" effort="10" velocity="1.0" />
   </joint>
   <link name="L2">
@@ -91,5 +91,5 @@
       <child link="L2" />
       <axis xyz="0 0 1" />
-      <limit lower="-1.57" upper="1.57" effort="0" velocity="0" />
+      <limit lower="-1.57" upper="1.57" effort="10" velocity="1.0" />
   </joint>
   <link name="L3">
@@ -121,5 +121,5 @@
       <child link="L3" />
       <axis xyz="0 0 -1" />
-      <limit lower="-1.57" upper="1.57" effort="0" velocity="0" />
+      <limit lower="-1.57" upper="1.57" effort="10" velocity="1.0" />
   </joint>
   <link name="L4">
@@ -150,5 +150,5 @@
       <child link="L4" />
       <axis xyz="0 0 1" />
-      <limit lower="-1.57" upper="1.57" effort="0" velocity="0" />
+      <limit lower="-1.57" upper="1.57" effort="10" velocity="1.0" />
   </joint>
   <link name="L5">
@@ -180,5 +180,5 @@
       <child link="L5" />
       <axis xyz="0 0 -1" />
-        <limit lower="-1.57" upper="1.57" effort="0" velocity="0" />
+        <limit lower="-1.57" upper="1.57" effort="10" velocity="1.0" />
   </joint>
   <link name="L6">
@@ -210,5 +210,5 @@
       <child link="L6" />
       <axis xyz="0 0 -1" />
-      <limit lower="0" upper="0" effort="0" velocity="0" />
+      <limit lower="-1.57" upper="1.57" effort="10" velocity="1.0" />
   </joint>
   <link name="suction_gripper">
