Commit message: Changed mesh file path

File: parol6_description/urdf/parol6_base.urdf.xacro (robot description, xacro)
@@ -16,11 +16,11 @@
         <origin xyz="0 0 0" rpy="0 0 0" />
         <geometry>
-          <mesh filename="file:///home/azif/projetcs/parol6/parol6_description/meshes/base_link.dae"/>
-        </geometry>
-      </visual>
-      <collision>
-        <origin xyz="0 0 0" rpy="0 0 0" />
-        <geometry>
-          <mesh filename="file:///home/azif/projetcs/parol6/parol6_description/meshes/base_link.dae"/>
+          <mesh filename="package://parol6_description/meshes/base_link.STL"/>
+        </geometry>
+      </visual>
+      <collision>
+        <origin xyz="0 0 0" rpy="0 0 0" />
+        <geometry>
+          <mesh filename="package://parol6_description/meshes/base_link.STL"/>
         </geometry>
       </collision>
@@ -40,11 +40,11 @@
         <origin xyz="0 0 0" rpy="0 0 0" />
         <geometry>
-          <mesh filename="file:///home/azif/projetcs/parol6/parol6_description/meshes/L1.dae"/>
-        </geometry>
-      </visual>
-      <collision>
-        <origin xyz="0 0 0" rpy="0 0 0" />
-        <geometry>
-          <mesh filename="file:///home/azif/projetcs/parol6/parol6_description/meshes/L1.dae"/>
+          <mesh filename="package://parol6_description/meshes/L1.STL"/>
+        </geometry>
+      </visual>
+      <collision>
+        <origin xyz="0 0 0" rpy="0 0 0" />
+        <geometry>
+          <mesh filename="package://parol6_description/meshes/L1.STL"/>
         </geometry>
       </collision>
@@ -67,11 +67,11 @@
         <origin xyz="0 0 0" rpy="0 0 0" />
         <geometry>
-          <mesh filename="file:///home/azif/projetcs/parol6/parol6_description/meshes/L2.dae"/>
-        </geometry>
-      </visual>
-      <collision>
-        <origin xyz="0 0 0" rpy="0 0 0" />
-        <geometry>
-          <mesh filename="file:///home/azif/projetcs/parol6/parol6_description/meshes/L2.dae"/>
+          <mesh filename="package://parol6_description/meshes/L2.STL"/>
+        </geometry>
+      </visual>
+      <collision>
+        <origin xyz="0 0 0" rpy="0 0 0" />
+        <geometry>
+          <mesh filename="package://parol6_description/meshes/L2.STL"/>
         </geometry>
       </collision>
@@ -94,11 +94,11 @@
         <origin xyz="0 0 0" rpy="0 0 0" />
         <geometry>
-          <mesh filename="file:///home/azif/projetcs/parol6/parol6_description/meshes/L3.dae"/>
-        </geometry>
-      </visual>
-      <collision>
-        <origin xyz="0 0 0" rpy="0 0 0" />
-        <geometry>
-          <mesh filename="file:///home/azif/projetcs/parol6/parol6_description/meshes/L3.dae"/>
+          <mesh filename="package://parol6_description/meshes/L3.STL"/>
+        </geometry>
+      </visual>
+      <collision>
+        <origin xyz="0 0 0" rpy="0 0 0" />
+        <geometry>
+          <mesh filename="package://parol6_description/meshes/L3.STL"/>
         </geometry>
       </collision>
@@ -121,10 +121,10 @@
         <origin xyz="0 0 0" rpy="0 0 0" />
         <geometry>
-          <mesh filename="file:///home/azif/projetcs/parol6/parol6_description/meshes/L4.dae"/>
-        </geometry>
-      </visual>
-      <collision>
-        <geometry>
-           <mesh filename="file:///home/azif/projetcs/parol6/parol6_description/meshes/L4.dae"/>
+          <mesh filename="package://parol6_description/meshes/L4.STL"/>
+        </geometry>
+      </visual>
+      <collision>
+        <geometry>
+           <mesh filename="package://parol6_description/meshes/L4.STL"/>
         </geometry>
       </collision>
@@ -152,5 +152,5 @@
       <origin xyz="0 0 0" rpy="0 0 0" />
       <geometry>
-        <mesh filename="file:///home/azif/projetcs/parol6/parol6_description/meshes/L5.dae"/>
+        <mesh filename="package://parol6_description/meshes/L5.STL"/>
       </geometry>
     </visual>
@@ -158,5 +158,5 @@
       <origin xyz="0 0 0" rpy="0 0 0" />
       <geometry>
-        <mesh filename="file:///home/azif/projetcs/parol6/parol6_description/meshes/L5.dae"/>
+        <mesh filename="package://parol6_description/meshes/L5.STL"/>
       </geometry>
     </collision>
@@ -184,5 +184,5 @@
       <origin xyz="0 0 0" rpy="0 0 0" />
       <geometry>
-        <mesh filename="file:///home/azif/projetcs/parol6/parol6_description/meshes/vaccum_gripper_holder.stl"/>
+        <mesh filename="package://parol6_description/meshes/vaccum_gripper_holder.stl"/>
       </geometry>
     </visual>
@@ -190,5 +190,5 @@
       <origin xyz="0 0 0" rpy="0 0 0" />
       <geometry>
-        <mesh filename="file:///home/azif/projetcs/parol6/parol6_description/meshes/vaccum_gripper_holder.stl"/>
+        <mesh filename="package://parol6_description/meshes/vaccum_gripper_holder.stl"/>
       </geometry>
     </collision>
@@ -205,5 +205,5 @@
       <origin xyz="0 0 0" rpy="0 0 0"/>
       <geometry>
-        <mesh filename="file:///home/azif/projetcs/parol6/parol6_description/meshes/vaccum_gripper.stl"/>
+        <mesh filename="package://parol6_description/meshes/vaccum_gripper.stl"/>
       </geometry>
     </visual>
@@ -211,5 +211,5 @@
       <origin xyz="0 0 0" rpy="0 0 0"/>
       <geometry>
-        <mesh filename="file:///home/azif/projetcs/parol6/parol6_description/meshes/vaccum_gripper.stl"/>
+        <mesh filename="package://parol6_description/meshes/vaccum_gripper.stl"/>
       </geometry>
     </collision>

Commit message: Add initial implementation of parol6_gui for controlling the Parol6 robot
- Created .gitignore to exclude build artifacts and temporary files.
- Added CMakeLists.txt for project configuration and dependencies.
- Implemented main application entry point in main.cpp.
- Developed MainWindow class with UI and ROS 2 integration in mainwindow.cpp and mainwindow.h.
- Designed UI layout in mainwindow.ui for controlling robot joints and targets.
- Included package.xml for ROS 2 package metadata and dependencies.

File: parol6_description/urdf/parol6_base.urdf.xacro (robot description, xacro)
@@ -6,5 +6,5 @@
 <robot xmlns:xacro="http://wiki.ros.org/xacro"
       name="parol6">
-    <link name="base_link">
+  <link name="base_link">
       <inertial>
         <origin xyz="-0.0274562034602567 -0.00137265400595656 0.031237920982338" rpy="0 0 0" />
@@ -25,10 +25,13 @@
         </geometry>
       </collision>
-    </link>
-    <!-- <gazebo reference="base_link">
+  </link>
+  <!-- <gazebo reference="base_link>
       <material>Gazebo/Orange</material>
       <turnGravityOff>false</turnGravityOff>
-    </gazebo> -->
-    <link name="L1">
+  </gazebo> -->
+  <gazebo reference="base_link">
+      <material>Gazebo/Grey</material>
+  </gazebo>
+  <link name="L1">
       <inertial>
         <origin xyz="0.00524529891406311 0.0289722820784871 0.0992791429452917" rpy="0 0 0" />
@@ -49,6 +52,9 @@
         </geometry>
       </collision>
-    </link>
-    <joint name="J1" type="revolute">
+  </link>
+  <gazebo reference="L1">
+      <material>Gazebo/Grey</material>
+  </gazebo>
+  <joint name="J1" type="revolute">
       <origin xyz="0 0 0" rpy="0 0 0" />
       <parent link="base_link" />
@@ -56,6 +62,6 @@
       <axis xyz="0 0 1" />
       <limit lower="-3.14" upper="3.14" effort="0" velocity="0" />
-    </joint>
-    <link name="L2">
+  </joint>
+  <link name="L2">
       <inertial>
         <origin xyz="-0.0094181617193695 -0.0783879603613605 0.0369429741417731" rpy="0 0 0" />
@@ -76,6 +82,9 @@
         </geometry>
       </collision>
-    </link>
-    <joint name="J2" type="revolute">
+  </link>
+  <gazebo reference="L2">
+      <material>Gazebo/Grey</material>
+  </gazebo>
+  <joint name="J2" type="revolute">
       <origin xyz="0.0234207210610375 0 0.1105" rpy="-1.5707963267949 0 0" />
       <parent link="L1" />
@@ -83,6 +92,6 @@
       <axis xyz="0 0 1" />
       <limit lower="-1.57" upper="1.57" effort="0" velocity="0" />
-    </joint>
-    <link name="L3">
+  </joint>
+  <link name="L3">
       <inertial>
         <origin xyz="0.0155509885239593 -0.0191127686426613 -0.00153322577917236" rpy="0 0 0" />
@@ -103,6 +112,9 @@
         </geometry>
       </collision>
-    </link>
-    <joint name="J3" type="revolute">
+  </link>
+  <gazebo reference="L3">
+      <material>Gazebo/Grey</material>
+  </gazebo>
+  <joint name="J3" type="revolute">
       <origin xyz="0 -0.18 0" rpy="3.1416 0 -1.5708" />
       <parent link="L2" />
@@ -110,6 +122,6 @@
       <axis xyz="0 0 -1" />
       <limit lower="-1.57" upper="1.57" effort="0" velocity="0" />
-    </joint>
-    <link name="L4">
+  </joint>
+  <link name="L4">
       <inertial>
         <origin xyz="0.000947028430634433 -0.008978947112462 -0.0924798659827059" rpy="0 0 0" />
@@ -129,6 +141,9 @@
         </geometry>
       </collision>
-    </link>
-    <joint name="J4" type="revolute">
+  </link>
+  <gazebo reference="L4">
+      <material>Gazebo/Grey</material>
+  </gazebo>
+  <joint name="J4" type="revolute">
       <origin xyz="0.0435 0.0 0.0" rpy="1.5708 0 3.1415" />
       <parent link="L3" />
@@ -136,101 +151,113 @@
       <axis xyz="0 0 1" />
       <limit lower="-1.57" upper="1.57" effort="0" velocity="0" />
-    </joint>
-    <link name="L5">
-    <inertial>
-      <origin xyz="6.7162171684676E-06 -0.00621420980825221 -0.000960871025916146" rpy="0 0 0" />
-      <mass value="0.185171777001718" />
-      <inertia
-        ixx="0.000109176748460021"
-        ixy="-1.27195013439061E-07"
-        ixz="8.4436049148633E-08"
-        iyy="8.41307588934268E-05"
-        iyz="-4.41596193640049E-07"
-        izz="0.000110629136236229" />
-    </inertial>
-    <visual>
-      <origin xyz="0 0 0" rpy="0 0 0" />
-      <geometry>
-        <mesh filename="package://parol6_description/meshes/L5.STL"/>
-      </geometry>
-    </visual>
-    <collision>
-      <origin xyz="0 0 0" rpy="0 0 0" />
-      <geometry>
-        <mesh filename="package://parol6_description/meshes/L5.STL"/>
-      </geometry>
-    </collision>
-  </link>
+  </joint>
+  <link name="L5">
+      <inertial>
+        <origin xyz="6.7162171684676E-06 -0.00621420980825221 -0.000960871025916146" rpy="0 0 0" />
+        <mass value="0.185171777001718" />
+        <inertia
+          ixx="0.000109176748460021"
+          ixy="-1.27195013439061E-07"
+          ixz="8.4436049148633E-08"
+          iyy="8.41307588934268E-05"
+          iyz="-4.41596193640049E-07"
+          izz="0.000110629136236229" />
+      </inertial>
+      <visual>
+        <origin xyz="0 0 0" rpy="0 0 0" />
+        <geometry>
+          <mesh filename="package://parol6_description/meshes/L5.STL"/>
+        </geometry>
+      </visual>
+      <collision>
+        <origin xyz="0 0 0" rpy="0 0 0" />
+        <geometry>
+          <mesh filename="package://parol6_description/meshes/L5.STL"/>
+        </geometry>
+      </collision>
+  </link>
+  <gazebo reference="L5">
+      <material>Gazebo/Grey</material>
+  </gazebo>
   <joint name="J5" type="revolute">
-    <origin xyz="0 0 -0.17635" rpy="-1.5708 0 0" />
-    <parent link="L4" />
-    <child link="L5" />
-    <axis xyz="0 0 -1" />
-      <limit lower="-1.57" upper="1.57" effort="0" velocity="0" />
+      <origin xyz="0 0 -0.17635" rpy="-1.5708 0 0" />
+      <parent link="L4" />
+      <child link="L5" />
+      <axis xyz="0 0 -1" />
+        <limit lower="-1.57" upper="1.57" effort="0" velocity="0" />
   </joint>
   <link name="L6">
-    <inertial>
-      <origin xyz="0.00632955087228015 -0.000453856352095022 -0.0554441567386594" rpy="0 0 0" />
-      <mass value="0.0703261410665101" />
-      <inertia
-        ixx="1.40276237518287E-05"
-        ixy="3.15503246005279E-07"
-        ixz="-9.28469598788221E-07"
-        iyy="1.81406721166117E-05"
-        iyz="-9.43630009030796E-07"
-        izz="2.34608103291027E-05" />
-    </inertial>
-    <visual>
-      <origin xyz="0 0 0" rpy="0 0 0" />
-      <geometry>
-        <mesh filename="package://parol6_description/meshes/vaccum_gripper_holder.stl"/>
-      </geometry>
-    </visual>
-    <collision>
-      <origin xyz="0 0 0" rpy="0 0 0" />
-      <geometry>
-        <mesh filename="package://parol6_description/meshes/vaccum_gripper_holder.stl"/>
-      </geometry>
-    </collision>
-  </link>
+      <inertial>
+        <origin xyz="0.00632955087228015 -0.000453856352095022 -0.0554441567386594" rpy="0 0 0" />
+        <mass value="0.0703261410665101" />
+        <inertia
+          ixx="1.40276237518287E-05"
+          ixy="3.15503246005279E-07"
+          ixz="-9.28469598788221E-07"
+          iyy="1.81406721166117E-05"
+          iyz="-9.43630009030796E-07"
+          izz="2.34608103291027E-05" />
+      </inertial>
+      <visual>
+        <origin xyz="0 0 0" rpy="0 0 0" />
+        <geometry>
+          <mesh filename="package://parol6_description/meshes/vaccum_gripper_holder.stl"/>
+        </geometry>
+      </visual>
+      <collision>
+        <origin xyz="0 0 0" rpy="0 0 0" />
+        <geometry>
+          <mesh filename="package://parol6_description/meshes/vaccum_gripper_holder.stl"/>
+        </geometry>
+      </collision>
+  </link>
+  <gazebo reference="L6">
+      <material>Gazebo/Orange</material>
+  </gazebo>
   <joint name="J6" type="continuous">
-    <origin xyz="0 0 0" rpy="1.5708 0 0" />
-    <parent link="L5" />
-    <child link="L6" />
-    <axis xyz="0 0 -1" />
-    <limit lower="0" upper="0" effort="0" velocity="0" />
+      <origin xyz="0 0 0" rpy="1.5708 0 0" />
+      <parent link="L5" />
+      <child link="L6" />
+      <axis xyz="0 0 -1" />
+      <limit lower="0" upper="0" effort="0" velocity="0" />
   </joint>
   <link name="suction_gripper">
-    <visual>
+      <visual>
+        <origin xyz="0 0 0" rpy="0 0 0"/>
+        <geometry>
+          <mesh filename="package://parol6_description/meshes/vaccum_gripper.stl"/>
+        </geometry>
+      </visual>
+      <collision>
+        <origin xyz="0 0 0" rpy="0 0 0"/>
+        <geometry>
+          <mesh filename="package://parol6_description/meshes/vaccum_gripper.stl"/>
+        </geometry>
+      </collision>
+      <inertial>
+        <origin xyz="0 0 0" rpy="0 0 0"/>
+        <mass value="0.01"/>
+        <inertia
+          ixx="1e-6" ixy="0" ixz="0"
+          iyy="1e-6" iyz="0"
+          izz="1e-6"/>
+      </inertial>
+  </link>
+  <gazebo reference="suction_gripper">
+      <material>Gazebo/Orange</material>
+  </gazebo>
+  <joint name="J7" type="fixed">
+      <parent link="L6"/>
+      <child link="suction_gripper"/>
       <origin xyz="0 0 0" rpy="0 0 0"/>
-      <geometry>
-        <mesh filename="package://parol6_description/meshes/vaccum_gripper.stl"/>
-      </geometry>
-    </visual>
-    <collision>
-      <origin xyz="0 0 0" rpy="0 0 0"/>
-      <geometry>
-        <mesh filename="package://parol6_description/meshes/vaccum_gripper.stl"/>
-      </geometry>
-    </collision>
-    <inertial>
-      <origin xyz="0 0 0" rpy="0 0 0"/>
-      <mass value="0.01"/>
-      <inertia
-        ixx="1e-6" ixy="0" ixz="0"
-        iyy="1e-6" iyz="0"
-        izz="1e-6"/>
-    </inertial>
-  </link>
-  <joint name="J7" type="fixed">
-    <parent link="L6"/>
-    <child link="suction_gripper"/>
-    <origin xyz="0 0 0" rpy="0 0 0"/>
   </joint>
   <link name="tool0"/>
+  <gazebo reference="tool0">
+      <material>Gazebo/Yellow</material>
+  </gazebo>
   <joint name="tool0_fixed" type="fixed">
-    <parent link="suction_gripper"/>
-    <child link="tool0"/>
-    <origin xyz="0.083695 -0.000779 -0.060305" rpy="0 0 0"/>
+      <parent link="suction_gripper"/>
+      <child link="tool0"/>
+      <origin xyz="0.083695 -0.000779 -0.060305" rpy="0 0 0"/>
   </joint>
 </robot>
