Commit message: Refactor box detector and GUI integration
- Changed joint type from continuous to revolute in URDF for J6.
- Added subscription to "/detected_box_info" in the GUI to display detected box information.
- Updated the box detector to publish box detection information and pose.
- Improved detection logic in box_detector.cpp, including RANSAC for plane fitting and enhanced box detection criteria.
- Added parameters for square tolerance and plane inlier threshold in box detection.
- Enhanced visualization and logging for detected boxes in the GUI.

File: parol6_description/urdf/parol6_base.urdf.xacro (robot description, xacro)
@@ -205,5 +205,5 @@
       <material>Gazebo/Orange</material>
   </gazebo>
-  <joint name="J6" type="continuous">
+  <joint name="J6" type="revolute">
       <origin xyz="0.0 0.0 0.0" rpy="1.5708 0 0" />
       <parent link="L5" />

Commit message: Update box mass and increase joint velocity limits for improved performance

File: parol6_description/urdf/parol6_base.urdf.xacro (robot description, xacro)
@@ -61,5 +61,5 @@
       <child link="L1" />
       <axis xyz="0 0 1" />
-      <limit lower="-3.14" upper="3.14" effort="10" velocity="1.0" />
+      <limit lower="-3.14" upper="3.14" effort="10" velocity="2.0" />
   </joint>
   <link name="L2">
@@ -91,5 +91,5 @@
       <child link="L2" />
       <axis xyz="0 0 1" />
-      <limit lower="-1.57" upper="1.57" effort="10" velocity="1.0" />
+      <limit lower="-1.57" upper="1.57" effort="10" velocity="2.0" />
   </joint>
   <link name="L3">
@@ -121,5 +121,5 @@
       <child link="L3" />
       <axis xyz="0 0 -1" />
-      <limit lower="-1.57" upper="1.57" effort="10" velocity="1.0" />
+      <limit lower="-1.57" upper="1.57" effort="10" velocity="2.0" />
   </joint>
   <link name="L4">
@@ -150,5 +150,5 @@
       <child link="L4" />
       <axis xyz="0 0 1" />
-      <limit lower="-1.57" upper="1.57" effort="10" velocity="1.0" />
+      <limit lower="-1.57" upper="1.57" effort="10" velocity="2.0" />
   </joint>
   <link name="L5">
@@ -180,5 +180,5 @@
       <child link="L5" />
       <axis xyz="0 0 -1" />
-        <limit lower="-1.57" upper="1.57" effort="10" velocity="1.0" />
+        <limit lower="-1.57" upper="1.57" effort="10" velocity="2.0" />
   </joint>
   <link name="L6">
@@ -210,5 +210,5 @@
       <child link="L6" />
       <axis xyz="0 0 -1" />
-      <limit lower="-1.57" upper="1.57" effort="10" velocity="1.0" />
+      <limit lower="-1.57" upper="1.57" effort="10" velocity="2.0" />
   </joint>
   <link name="suction_gripper">
